File: layout/g5500-ethernet-controller.sch (KiCad schematic (older format))
At the start: 18 parts, among them K1 G5LE-1, K2 G5LE-1, K3 G5LE-1, K4 G5LE-1, U1 NUCLEO144-F429ZI

Commit message: layout: Schematic poking, drag in components used in etherswitch.
Parts:
- removed C?: C, symbol agg-kicad:C
- removed D?: MB4S, Package_TO_SOT_SMD:TO-269AA, symbol Diode_Bridge:MB4S
- removed J?: CONN_01x03, symbol agg-kicad:CONN_01x03
- removed J?: CONN_01x02, symbol agg-kicad:CONN_01x02
- removed J?: MICROUSB, agg:MICROUSB_MOLEX_47589-0001, symbol agg-kicad:MICROUSB
- removed R?: R, symbol agg-kicad:R
- removed U?: TSR_1-2450, Converters_DCDC_ACDC:DCDC-Conv_TRACO_TSR-1, symbol Regulator_Switching:TSR_1-2450
- added C? (x5): 2u2, symbol agg-kicad:C
- added D? (x4): MBR0580, Diode_SMD:D_SOD-123, symbol Diode:MBR0580
- added J?: CONN_01x03, symbol agg-kicad:CONN_01x03
- added Q?: BC817W, Package_TO_SOT_SMD:SOT-323_SC-70, symbol Transistor_BJT:BC817W
- added R? (x2): 10K, symbol agg-kicad:R
- added R?: 100R, symbol agg-kicad:R
- added R?: 1K, symbol agg-kicad:R
- C?: value C -> 2u2
- R?: value R -> 100R
Connections:
- net labels added: 3v3, GND, STM_AZ_ANALOG, STM_AZ_CCW, STM_AZ_CW, STM_EL_ANALOG, STM_EL_DN, STM_EL_UP
- wire segments 71 -> 103
Other:
- moved on the sheet: R?

Commit message: Progress on layout.
Parts:
- added C10, C11, C13, C17, C8, C9: 2u2, agg:0603, symbol agg-kicad:C
- added C12: 0.1u, agg:0603, symbol agg-kicad:C
- added C14, C7: 100n, agg:0603, symbol agg-kicad:C
- added C15: 100p, agg:0603, symbol agg-kicad:C
- added C16, C18: 10n, agg:0402, symbol agg-kicad:C
- added C19: 0F22, Capacitor_THT:C_Rect_L11.5mm_W9.8mm_P10.00mm_MKT, symbol agg-kicad:C
- added D5: LED, agg:0603-LED, symbol agg-kicad:LED
- added D6: D, Diode_SMD:D_SOD-123, symbol agg-kicad:D
- added IC1: MAX-M8Q, agg:MAX-M8Q, symbol agg-kicad:MAX-M8Q
- added J3: MICROUSB, agg:MICROUSB_MOLEX_47589-0001, symbol agg-kicad:MICROUSB
- added L1: 27n, agg:0402, symbol agg-kicad:L
- added P1: COAX, agg:SMA-EDGE, symbol agg-kicad:COAX
- added Q2, Q3, Q4: BC817W, Package_TO_SOT_SMD:SOT-323_SC-70, symbol Transistor_BJT:BC817W
- added R10: 10R, agg:0402, symbol agg-kicad:R
- added R11, R12: 220R, agg:0603, symbol agg-kicad:R
- added R13: DNF, agg:0603, symbol agg-kicad:R
- added R14, R6, R7, R8: 1K, agg:0603, symbol agg-kicad:R
- added R9: R, agg:0603, symbol agg-kicad:R
- added U2: LD3985G33R_TSOT23, Package_TO_SOT_SMD:TSOT-23-5, symbol Regulator_Linear:LD3985G33R_TSOT23
- C1, C2, C3, C4, C5, C6: renamed from C?; footprint (none) -> agg:0603
- J1, J2, J5, J6: renamed from J?; footprint (none) -> Connector_Molex:Molex_KK-254_AE-6410-03A_1x03_P2.54mm_Vertical
- J4: renamed from J?; footprint (none) -> Connector_Molex:Molex_KK-254_AE-6410-02A_1x02_P2.54mm_Vertical
- R1, R2, R3, R4, R5: renamed from R?; footprint (none) -> agg:0603
- gave numbers to parts that had none: 5
Connections:
- net labels added: 5v, GPS_3V3, GPS_RXD, GPS_TXD, RELAY_CCW, RELAY_CW, RELAY_DOWN, RELAY_UP, VCC_RELAY
- wire segments 103 -> 231
Other:
- note added: "Actually TPS79933DDCR, but pinout matches."
- moved on the sheet: Q1, R5

Commit message: Layout nearly done.
Parts:
- added D10, D7, D8, D9: LED, agg:0603-LED, symbol agg-kicad:LED
- added J10, J9: CONN_01x03, Connector_Molex:Molex_KK-254_AE-6410-03A_1x03_P2.54mm_Vertical, symbol agg-kicad:CONN_01x03
- added J11, J7, J8: CONN_01x02, Connector_Molex:Molex_KK-254_AE-6410-02A_1x02_P2.54mm_Vertical, symbol agg-kicad:CONN_01x02
- added R15, R16, R17, R18: 1K, agg:0603, symbol agg-kicad:R
- C13: footprint agg:0603 -> Capacitor_SMD:C_0603_1608Metric
Connections:
- net labels added: AZ_CCW_SWITCH, AZ_CW_SWITCH, AZ_METER, EL_DN_SWITCH, EL_METER, EL_UP_SWITCH, ENABLE_SWITCH
- wire segments 231 -> 263

Commit message: layout: Finish and send off v1.
Parts:
- added R19, R22: 1K, agg:0603, symbol agg-kicad:R
- added R20, R21: 22R, agg:0603, symbol agg-kicad:R
- C13: footprint Capacitor_SMD:C_0603_1608Metric -> agg:0603
- R1, R2: value 100R -> 22R
Connections:
- wire segments 263 -> 267
Other:
- moved on the sheet: J1, J2
Changed lines of the file:
@@
 L agg-kicad:CONN_01x03 J2
 U 1 1 5A89F92A
-P 1680 7890
-F 0 "J2" H 1711 8105 50  0000 C CNN
-F 1 "CONN_01x03" H 1711 8014 50  0000 C CNN
-F 2 "Connector_Molex:Molex_KK-254_AE-6410-03A_1x03_P2.54mm_Vertical" H 1680 7890 50  0001 C CNN
-F 3 "" H 1680 7890 50  0001 C CNN
-	1    1680 7890
+P 1570 7890
+F 0 "J2" H 1601 8105 50  0000 C CNN
+F 1 "CONN_01x03" H 1601 8014 50  0000 C CNN
+F 2 "Connector_Molex:Molex_KK-254_AE-6410-03A_1x03_P2.54mm_Vertical" H 1570 7890 50  0001 C CNN
+F 3 "" H 1570 7890 50  0001 C CNN
+	1    1570 7890
 	1    0    0    -1
 $EndComp
@@
 P 1950 7890
 F 0 "R2" H 2000 8068 50  0000 C CNN
-F 1 "100R" H 2000 7977 50  0000 C CNN
+F 1 "22R" H 2000 7977 50  0000 C CNN
 F 2 "agg:0603" H 1950 7890 50  0001 C CNN
 F 3 "" H 1950 7890 50  0001 C CNN
@@
 Wire Wire Line
 	1880 7890 1880 8020
-Connection ~ 1880 7890
-Wire Wire Line
-	1880 7890 1780 7890
 Wire Wire Line
 	1810 8090 1810 8120
@@
 Connection ~ 2120 8120
 Wire Wire Line
-	1780 7990 2120 7990
-Wire Wire Line
 	2120 7990 2120 8020
 Wire Wire Line
 	2120 7990 2210 7990
-Connection ~ 2120 7990
 Wire Wire Line
 	2310 7990 2390 7990
@@
 L agg-kicad:CONN_01x03 J1
 U 1 1 5A8FB849
-P 1680 7310
-F 0 "J1" H 1711 7525 50  0000 C CNN
-F 1 "CONN_01x03" H 1711 7434 50  0000 C CNN
-F 2 "Connector_Molex:Molex_KK-254_AE-6410-03A_1x03_P2.54mm_Vertical" H 1680 7310 50  0001 C CNN
-F 3 "" H 1680 7310 50  0001 C CNN
-	1    1680 7310
+P 1570 7310
+F 0 "J1" H 1601 7525 50  0000 C CNN
+F 1 "CONN_01x03" H 1601 7434 50  0000 C CNN
+F 2 "Connector_Molex:Molex_KK-254_AE-6410-03A_1x03_P2.54mm_Vertical" H 1570 7310 50  0001 C CNN
+F 3 "" H 1570 7310 50  0001 C CNN
+	1    1570 7310
 	1    0    0    -1
 $EndComp
@@
 P 1950 7310
 F 0 "R1" H 2000 7488 50  0000 C CNN
-F 1 "100R" H 2000 7397 50  0000 C CNN
+F 1 "22R" H 2000 7397 50  0000 C CNN
 F 2 "agg:0603" H 1950 7310 50  0001 C CNN
 F 3 "" H 1950 7310 50  0001 C CNN
@@
 Wire Wire Line
 	1880 7310 1880 7440
-Connection ~ 1880 7310
-Wire Wire Line
-	1880 7310 1780 7310
 Wire Wire Line
 	1810 7510 1810 7540
@@
 Connection ~ 2120 7540
 Wire Wire Line
-	1780 7410 2120 7410
-Wire Wire Line
 	2120 7410 2120 7440
 Wire Wire Line
 	2120 7410 2210 7410
-Connection ~ 2120 7410
 Wire Wire Line
 	2310 7410 2390 7410
@@
 F 0 "C13" V 1844 4338 50  0000 L CNN
 F 1 "2u2" V 1935 4338 50  0000 L CNN
-F 2 "Capacitor_SMD:C_0603_1608Metric" H 1840 4280 50  0001 C CNN
+F 2 "agg:0603" H 1840 4280 50  0001 C CNN
 F 3 "" H 1840 4280 50  0001 C CNN
 	1    1840 4280
@@
 Connection ~ 1840 4250
 Wire Wire Line
-	1780 7510 1810 7510
-Wire Wire Line
-	1780 8090 1810 8090
+	1670 7510 1810 7510
+Wire Wire Line
+	1670 8090 1810 8090
 $Comp
 L agg-kicad:CONN_01x02 J7
@@
 Wire Wire Line
 	11410 2940 11410 2930
+$Comp
+L agg-kicad:R R21
+U 1 1 5AC4E62C
+P 1730 7890
+F 0 "R21" H 1780 8068 50  0000 C CNN
+F 1 "22R" H 1780 7977 50  0000 C CNN
+F 2 "agg:0603" H 1730 7890 50  0001 C CNN
+F 3 "" H 1730 7890 50  0001 C CNN
+	1    1730 7890
+	1    0    0    -1
+$EndComp
+Wire Wire Line
+	1880 7890 1830 7890
+Connection ~ 1880 7890
+Wire Wire Line
+	1730 7890 1670 7890
+$Comp
+L agg-kicad:R R22
+U 1 1 5AC9E76C
+P 1730 7990
+F 0 "R22" H 1780 8168 50  0000 C CNN
+F 1 "1K" H 1780 8077 50  0000 C CNN
+F 2 "agg:0603" H 1730 7990 50  0001 C CNN
+F 3 "" H 1730 7990 50  0001 C CNN
+	1    1730 7990
+	1    0    0    -1
+$EndComp
+Wire Wire Line
+	1830 7990 2120 7990
+Connection ~ 2120 7990
+Wire Wire Line
+	1730 7990 1670 7990
+$Comp
+L agg-kicad:R R20
+U 1 1 5AD197A9
+P 1730 7310
+F 0 "R20" H 1780 7488 50  0000 C CNN
+F 1 "22R" H 1780 7397 50  0000 C CNN
+F 2 "agg:0603" H 1730 7310 50  0001 C CNN
+F 3 "" H 1730 7310 50  0001 C CNN
+	1    1730 7310
+	1    0    0    -1
+$EndComp
+Wire Wire Line
+	1830 7310 1880 7310
+Connection ~ 1880 7310
+Wire Wire Line
+	1730 7310 1670 7310
+$Comp
+L agg-kicad:R R19
+U 1 1 5AD43024
+P 1720 7410
+F 0 "R19" H 1770 7588 50  0000 C CNN
+F 1 "1K" H 1770 7497 50  0000 C CNN
+F 2 "agg:0603" H 1720 7410 50  0001 C CNN
+F 3 "" H 1720 7410 50  0001 C CNN
+	1    1720 7410
+	1    0    0    -1
+$EndComp
+Wire Wire Line
+	1670 7410 1720 7410
+Wire Wire Line
+	1820 7410 2120 7410
+Connection ~ 2120 7410
 $EndSCHEMATC
